Commit message: modified:   config/ekf_localization.yaml 	modified:   description/imu.xacro 	modified:   description/robot_core.xacro

File: description/imu.xacro (robot description, xacro)
@@ -10,4 +10,58 @@
         <gravity>true</gravity>
         <sensor name="imu_sensor" type="imu">
+        <imu>
+          <angular_velocity>
+            <x>
+              <noise type="gaussian">
+                <mean>0.0</mean>
+                <stddev>2e-4</stddev>
+                <bias_mean>0.0000075</bias_mean>
+                <bias_stddev>0.0000008</bias_stddev>
+              </noise>
+            </x>
+            <y>
+              <noise type="gaussian">
+                <mean>0.0</mean>
+                <stddev>2e-4</stddev>
+                <bias_mean>0.0000075</bias_mean>
+                <bias_stddev>0.0000008</bias_stddev>
+              </noise>
+            </y>
+            <z>
+              <noise type="gaussian">
+                <mean>0.0</mean>
+                <stddev>2e-4</stddev>
+                <bias_mean>0.0000075</bias_mean>
+                <bias_stddev>0.0000008</bias_stddev>
+              </noise>
+            </z>
+          </angular_velocity>
+          <linear_acceleration>
+            <x>
+              <noise type="gaussian">
+                <mean>0.0</mean>
+                <stddev>1.7e-2</stddev>
+                <bias_mean>0.1</bias_mean>
+                <bias_stddev>0.001</bias_stddev>
+              </noise>
+            </x>
+            <y>
+              <noise type="gaussian">
+                <mean>0.0</mean>
+                <stddev>1.7e-2</stddev>
+                <bias_mean>0.1</bias_mean>
+                <bias_stddev>0.001</bias_stddev>
+              </noise>
+            </y>
+            <z>
+              <noise type="gaussian">
+                <mean>0.0</mean>
+                <stddev>1.7e-2</stddev>
+                <bias_mean>0.1</bias_mean>
+                <bias_stddev>0.001</bias_stddev>
+              </noise>
+            </z>
+          </linear_acceleration>
+        </imu>
         <always_on>true</always_on>
         <update_rate>100</update_rate>

File: description/robot_core.xacro (robot description, xacro)
@@ -25,5 +25,5 @@
     <xacro:property name="imu_x_offset_chassis" value="-0.03"/>
     <xacro:property name="imu_z_offset_chassis" value="0.0881"/>
-    <xacro:property name="friction_mu" value="5.0"/>
+    <xacro:property name="friction_mu" value="10000.0"/>
     <!-- Imports -->
     <xacro:include filename="inertial_macros.xacro"/>
