Commit message: modified:   description/laser.xacro 	modified:   scripts/figure_eight.py

File: description/laser.xacro (robot description, xacro)
@@ -8,5 +8,5 @@
     <link name="laser_frame">
         <visual>
-            <origin rpy="0 0 0" xyz="0 0 0.0141"/>
+            <origin rpy="0 0 ${pi}" xyz="0 0 0.0141"/>
             <geometry>
                 <mesh filename="package://astro/description/meshes/RPLidarA1.stl" scale="0.001 0.001 0.001"/>

Commit message: modified:   description/laser.xacro

File: description/laser.xacro (robot description, xacro)
@@ -4,9 +4,9 @@
         <parent link="chassis"/>
         <child link="laser_frame"/>
-        <origin xyz="${lidar_x_offset} 0 ${chassis_base_to_lidar_height}" rpy="0 0 0"/>
+        <origin xyz="${lidar_x_offset} 0 ${chassis_base_to_lidar_height}" rpy="0 0 ${pi}"/>
     </joint>
     <link name="laser_frame">
         <visual>
-            <origin rpy="0 0 ${pi}" xyz="0 0 0.0141"/>
+            <origin rpy="0 0 0" xyz="0 0 0.0141"/>
             <geometry>
                 <mesh filename="package://astro/description/meshes/RPLidarA1.stl" scale="0.001 0.001 0.001"/>

Commit message: modified:   CMakeLists.txt 	modified:   description/laser.xacro 	modified:   description/robot_core.xacro 	new file:   scripts/get_currents.py

File: description/laser.xacro (robot description, xacro)
@@ -8,5 +8,5 @@
     <link name="laser_frame">
         <visual>
-            <origin rpy="0 0 0" xyz="0 0 0.0141"/>
+            <origin rpy="0 0 ${pi}" xyz="0 0 0.0141"/>
             <geometry>
                 <mesh filename="package://astro/description/meshes/RPLidarA1.stl" scale="0.001 0.001 0.001"/>
@@ -15,5 +15,5 @@
         </visual>
         <collision>
-            <origin rpy="0 0 0" xyz="0 0 0.0141"/>
+            <origin rpy="0 0 ${pi}" xyz="0 0 0.0141"/>
             <geometry>
                 <mesh filename="package://astro/description/meshes/RPLidarA1.stl" scale="0.001 0.001 0.001"/>

File: description/robot_core.xacro (robot description, xacro)
@@ -11,5 +11,5 @@
     <xacro:property name="ground_clearance" value="0.0146"/>
     <xacro:property name="base_thickness" value="0.01"/>
-    <xacro:property name="chassis_mass" value="3.0"/>
+    <xacro:property name="chassis_mass" value="7.0"/>
     <xacro:property name="caster_wheel_mass" value="0.02"/>
     <xacro:property name="chassis_length" value="0.32"/>
