Commit message: renamed crta_diffbot -> astro 	modified:   CMakeLists.txt 	modified:   README.md 	renamed:    description/crta_diffbot.urdf.xacro -> description/astro.urdf.xacro 	modified:   description/laser.xacro 	modified:   description/robot_core.xacro 	modified:   launch/joy.launch 	modified:   launch/move_base.launch 	modified:   launch/navigation.launch 	modified:   launch/robot_bringup.launch 	modified:   launch/rsp.launch 	modified:   launch/save_map.launch 	modified:   launch/simulation.launch 	modified:   launch/start_gmapping.launch 	modified:   launch/start_slam.launch 	modified:   launch/twist_mux.launch 	modified:   package.xml

File: description/astro.urdf.xacro (robot description, xacro)
@@ -1,4 +1,4 @@
 <?xml version="1.0"?>
-<robot xmlns:xacro="http://www.ros.org/wiki/xacro"  name="crta_diffbot">
+<robot xmlns:xacro="http://www.ros.org/wiki/xacro"  name="astro">
     <xacro:include filename="robot_core.xacro" />
     <xacro:include filename="laser.xacro"/>

File: description/laser.xacro (robot description, xacro)
@@ -10,5 +10,5 @@
             <origin rpy="0 0 0" xyz="0 0 0.0141"/>
             <geometry>
-                <mesh filename="package://crta_diffbot/description/meshes/RPLidarA1.stl" scale="0.001 0.001 0.001"/>
+                <mesh filename="package://astro/description/meshes/RPLidarA1.stl" scale="0.001 0.001 0.001"/>
             </geometry>
             <material name="dark_gray"/>
@@ -17,5 +17,5 @@
             <origin rpy="0 0 0" xyz="0 0 0.0141"/>
             <geometry>
-                <mesh filename="package://crta_diffbot/description/meshes/RPLidarA1.stl" scale="0.001 0.001 0.001"/>
+                <mesh filename="package://astro/description/meshes/RPLidarA1.stl" scale="0.001 0.001 0.001"/>
             </geometry>
         </collision>

File: description/robot_core.xacro (robot description, xacro)
@@ -38,5 +38,5 @@
             <origin rpy="0 0 0" xyz="0 0 0"/>
             <geometry>
-                <mesh filename="package://crta_diffbot/description/meshes/Chassis.stl" scale="0.001 0.001 0.001"/>
+                <mesh filename="package://astro/description/meshes/Chassis.stl" scale="0.001 0.001 0.001"/>
             </geometry>
             <material name="gray"/>
@@ -45,5 +45,5 @@
             <origin rpy="0 0 0" xyz="0 0 0"/>
             <geometry>
-                <mesh filename="package://crta_diffbot/description/meshes/Chassis.stl" scale="0.001 0.001 0.001"/>
+                <mesh filename="package://astro/description/meshes/Chassis.stl" scale="0.001 0.001 0.001"/>
             </geometry>
         </collision>

Commit message: modified:   description/astro.urdf.xacro 	new file:   description/meshes/Intel_RealSense_D435.stl 	new file:   description/realsense.xacro 	modified:   description/robot_core.xacro 	modified:   launch/simulation.launch 	new file:   rviz/realsense_robot.rviz

File: description/astro.urdf.xacro (robot description, xacro)
@@ -3,4 +3,5 @@
     <xacro:include filename="robot_core.xacro" />
     <xacro:include filename="laser.xacro"/>
+    <xacro:include filename="realsense.xacro"/>
     <xacro:include filename="gazebo_control.xacro"/>
 </robot>

File: description/robot_core.xacro (robot description, xacro)
@@ -16,4 +16,11 @@
     <xacro:property name="chassis_width" value="0.337"/>
     <xacro:property name="chassis_height" value="0.085"/>
+    <xacro:property name="chassis_inertial_offset_x" value="0.015"/>
+    <xacro:property name="realsense_x_offset" value="0.175"/>
+    <xacro:property name="realsense_z_offset_chassis" value="0.0425"/>
+    <xacro:property name="realsense_depth_offset" value="0.0175"/>
+    <xacro:property name="realsense_depth_to_infra1_offset" value="0.0"/>
+    <xacro:property name="realsense_depth_to_infra2_offset" value="-0.050"/>
+    <xacro:property name="realsense_depth_to_color_offset" value="0.015"/>
     <xacro:property name="friction_mu" value="10000"/>
     <!-- Imports -->
@@ -49,5 +56,5 @@
         </collision>
         <xacro:inertial_box mass="${chassis_mass}" x="${chassis_length}" y="${chassis_width}" z="${chassis_height}">
-            <origin xyz="0 0 ${chassis_height/2}" rpy="0 0 0"/>
+            <origin xyz="${chassis_inertial_offset_x} 0 ${chassis_height/2}" rpy="0 0 0"/>
         </xacro:inertial_box>
     </link>

Commit message: new file:   config/ekf_localization.yaml 	modified:   description/astro.urdf.xacro 	modified:   description/gazebo_control.xacro 	new file:   description/imu.xacro 	modified:   description/robot_core.xacro 	modified:   launch/navigation.launch 	modified:   launch/robot_bringup.launch 	modified:   launch/rsp.launch 	new file:   launch/sensor_fusion.launch 	modified:   launch/simulation.launch 	modified:   launch/start_gmapping.launch 	new file:   launch/start_hardware.launch 	modified:   launch/twist_mux.launch 	modified:   package.xml 	modified:   rviz/move_robot.rviz

File: description/astro.urdf.xacro (robot description, xacro)
@@ -4,4 +4,5 @@
     <xacro:include filename="laser.xacro"/>
     <xacro:include filename="realsense.xacro"/>
+    <xacro:include filename="imu.xacro"/>
     <xacro:include filename="gazebo_control.xacro"/>
 </robot>

File: description/gazebo_control.xacro (robot description, xacro)
@@ -12,10 +12,11 @@
             <torque>1000</torque>
             <commandTopic>cmd_vel</commandTopic>
-            <odometryTopic>odom</odometryTopic>
+            <odometryTopic>odom_raw</odometryTopic>
             <odometryFrame>odom</odometryFrame>
             <odometrySource>1</odometrySource>
             <robotBaseFrame>base_footprint</robotBaseFrame>
             <publishWheelTF>false</publishWheelTF>
-            <publishOdomTF>true</publishOdomTF>
+            <!-- publishOdomTF false if using sensor fusion (robot_localization), otherwise true -->
+            <publishOdomTF>false</publishOdomTF>
             <publishTf>1</publishTf>
             <wheelTorque>5</wheelTorque>

File: description/robot_core.xacro (robot description, xacro)
@@ -23,5 +23,7 @@
     <xacro:property name="realsense_depth_to_infra2_offset" value="-0.050"/>
     <xacro:property name="realsense_depth_to_color_offset" value="0.015"/>
-    <xacro:property name="friction_mu" value="10000"/>
+    <xacro:property name="imu_x_offset_chassis" value="-0.03"/>
+    <xacro:property name="imu_z_offset_chassis" value="0.0881"/>
+    <xacro:property name="friction_mu" value="5.0"/>
     <!-- Imports -->
     <xacro:include filename="inertial_macros.xacro"/>

Commit message: modified:   description/astro.urdf.xacro 	modified:   description/lidar.xacro 	modified:   description/materials.xacro 	new file:   description/realsense.xacro 	new file:   description/ros2_control.xacro 	new file:   launch/lidar.launch.py 	new file:   meshes/RealSense.dae 	modified:   package.xml 	new file:   rviz/view_lidar.rviz

File: description/astro.urdf.xacro (robot description, xacro)
@@ -3,3 +3,4 @@
     <xacro:include filename="robot_core.xacro" />
     <xacro:include filename="lidar.xacro"/>
+    <xacro:include filename="realsense.xacro"/>
 </robot>

File: description/lidar.xacro (robot description, xacro)
@@ -4,9 +4,9 @@
         <parent link="base_link"/>
         <child link="laser_frame"/>
-        <origin xyz="${lidar_x_offset} 0 ${lidar_z_offset - 0.0171}" rpy="0 0 0"/>
+        <origin xyz="${lidar_x_offset} 0 ${lidar_z_offset - 0.0171}" rpy="0 0 ${pi}"/>
     </joint>
     <link name="laser_frame">
         <visual>
-            <origin rpy="0 0 0" xyz="0 0 0.0171"/>
+            <origin rpy="0 0 ${pi}" xyz="0 0 0.0171"/>
             <geometry>
                 <mesh filename="package://astro/meshes/ASTRO_LidarAssembly.stl" scale="0.001 0.001 0.001"/>
@@ -15,5 +15,5 @@
         </visual>
         <collision>
-            <origin rpy="0 0 0" xyz="0 0 0.0171"/>
+            <origin rpy="0 0 ${pi}" xyz="0 0 0.0171"/>
             <geometry>
                 <mesh filename="package://astro/meshes/ASTRO_LidarAssembly.stl" scale="0.001 0.001 0.001"/>

File: description/materials.xacro (robot description, xacro)
@@ -22,3 +22,9 @@
         <color rgba="0.2 0.2 0.2 1"/>
     </material>
+    <material name="aluminum">
+        <color rgba="0.1 0.1 0.1 1"/>
+    </material>
+    <material name="plastic">
+        <color rgba="0.1 0.1 0.1 1"/>
+    </material>
 </robot>
